File: ESP32.kicad_sch (KiCad schematic)
At the start: 0 parts

Commit message: Liligo module added
Parts:
- added U1: T-Display-S3, esp32:T-Display-S3, symbol esp32:T-Display-S3
Connections:
- new net +3.3V: U1.1 (3v), U1.24 (3v)
- new net GND: U1.11 (GND), U1.13 (GND), U1.14 (GND), U1.22 (GND), U1.23 (GND)

Commit message: Big changes! DAC, ADC, ESP32
schematic 80% complete
added pcm libary part of module maybe someone can use it :)
Parts:
- added J2: Pedal 1, Connector_PinSocket_2.54mm:PinSocket_1x03_P2.54mm_Vertical, symbol Connector:Conn_01x03_Pin
Connections:
- net +3.3V: now also J2.3 (Pin_3)
- net GND: now also J2.1 (Pin_1)
- net 43: now reaches U1.15 (43)
- net 44: now reaches U1.16 (44)
- net 18/WS: now reaches U1.17 (18)
- net 17: now reaches U1.18 (17)
- net 21: now reaches U1.19 (21)
- net PB1: now reaches U1.2 (1)
- net PB1: now also J2.2 (Pin_2)
- net 16: now reaches U1.20 (16)
- net PB2: now reaches U1.3 (2)
- net PK1: now reaches U1.4 (3)
- net PB3: now reaches U1.5 (10)
- net PK2: now reaches U1.6 (11)
- net PK3: now reaches U1.7 (12)
- net PK4: now reaches U1.8 (13)

Commit message: PCB layout
schematic finished, layout
Parts:
- added C10, C11, C12, C13, C14, C15, C16, C9: 10nF, Capacitor_SMD:C_0805_2012Metric_Pad1.18x1.45mm_HandSolder, symbol Device:C
- added C17: 100 uF 16 V, Capacitor_THT:CP_Radial_D10.0mm_P5.00mm, symbol Device:C_Polarized
- added D1: Blue LED (5V), LED_THT:LED_D5.0mm, symbol Device:LED
- added D2: Blue LED (5VA), LED_THT:LED_D5.0mm, symbol Device:LED
- added D3: Green LED (3.3V), LED_THT:LED_D5.0mm, symbol Device:LED
- added J3, J4: SJ1-3525NG-PI, SamacSys_Parts:SJ13525NGPI, symbol SamacSys_Parts:SJ1-3525NG-PI
- added J6: Conn_02x01, Connector_PinHeader_2.54mm:PinHeader_2x01_P2.54mm_Vertical, symbol Connector_Generic:Conn_02x01
- added J7: Boot, Connector_PinHeader_2.54mm:PinHeader_2x01_P2.54mm_Vertical, symbol Connector_Generic:Conn_02x01
- added R5, R6, R7: 1k 0.25W, Resistor_THT:R_Axial_DIN0204_L3.6mm_D1.6mm_P5.08mm_Horizontal, symbol Device:R
- added SW2: SW_Push, Button_Switch_THT:SW_PUSH_6mm_H13mm, symbol Switch:SW_Push
- added SW3: Boot, Button_Switch_THT:SW_PUSH_6mm_H13mm, symbol Switch:SW_Push
- added VR1, VR2, VR3, VR4, VR5: RK09K1130AAU, SamacSys_Parts:RK09K1130AAU, symbol SamacSys_Parts:RK09K1130AAU
Connections:
- net +3.3V: now also J3.2 (TIP), J4.2 (TIP), R7.1, VR1.1 (CCW), VR2.1 (CCW), VR3.1 (CCW), VR4.1 (CCW), VR5.1 (CCW)
- net GND: now also C10.2, C11.2, C12.2, C13.2, C14.2, C15.2, C16.2, C17.2, C9.2, D1.1 (K), D2.1 (K), D3.1 (K), J3.1 (SLEEVE), J4.1 (SLEEVE), VR1.3 (CW), VR1.4 (MH_1), VR1.5 (MH_2), VR2.3 (CW), VR2.4 (MH_1), VR2.5 (MH_2), VR3.3 (CW), VR3.4 (MH_1), VR3.5 (MH_2), VR4.3 (CW), VR4.4 (MH_1), VR4.5 (MH_2), VR5.3 (CW), VR5.4 (MH_1), VR5.5 (MH_2)
- net PB1: now also C9.1
- net PB2: now also C10.1, J3.3 (RING)
- net PB3: now also C11.1, J4.3 (RING)
- net PK1: now also C12.1, VR1.2 (WIPER)
- net PK2: now also C13.1, VR2.2 (WIPER)
- net PK3: now also C14.1, VR3.2 (WIPER)
- net PK4: now also C15.1, VR4.2 (WIPER)
- net +5V: now reaches U1.12 (5V)
- net +5V: now also C17.1, R5.1
- net 16 renamed PK5
- net PK5: now also C16.1, VR5.2 (WIPER)
- new net: D3.2 (A), R7.2
- new net: D2.2 (A), R6.2
- new net: D1.2 (A), R5.2
- new net +5VA: R6.1
- new net Boot1: J7.2 (Pin_2), SW3.1
- new net Boot2: J7.1 (Pin_1), SW3.2
- new net Button1: J6.2 (Pin_2), SW2.1
- new net Button2: J6.1 (Pin_1), SW2.2
Other:
- note added: "Pedal 2"
- note added: "Pedal 3"
- note added: "Power Switch on the case, in series with the positive terminal of the battery It goes straight to the LilyGO board."
- moved on the sheet: J2
