File: Output.kicad_sch (KiCad schematic)
At the start: 0 parts

Commit message: Big changes! DAC, ADC, ESP32
schematic 80% complete
added pcm libary part of module maybe someone can use it :)
Parts:
- added J1: PCM5102A, Connector_PinSocket_2.54mm:PinSocket_1x11_P2.54mm_Vertical, symbol Connector:Conn_01x11_Socket
- added J4: Output 1/4", Connector_Audio:Jack_6.35mm_Neutrik_NRJ6HM-1-PRE_Horizontal, symbol Connector_Audio:AudioJack2_Ground_Switch
- added J5: PCM5102A_out, Connector_PinHeader_2.54mm:PinHeader_1x03_P2.54mm_Vertical, symbol Connector:Conn_01x03_Socket
- added SW1: SW_SP3T, Button_Switch_SMD:SW_SP3T_PCM13, symbol Switch:SW_SP3T
Connections:
- new net +5VA: J1.1 (Pin_1)
- new net BCK: J1.7 (Pin_7)
- new net DIN: J1.8 (Pin_8)
- new net GND: J1.10 (Pin_10), J1.3 (Pin_3), J1.4 (Pin_4), J1.5 (Pin_5), J1.6 (Pin_6), J4.G, J5.2 (Pin_2)
- new net LCK: J1.9 (Pin_9)
- new net OutputL: J4.T, J5.1 (Pin_1), SW1.1
- new net OutputR: J4.S, SW1.3
- new net PCMOutputR: J5.3 (Pin_3), SW1.2
- new net XMT/3V3: J1.11 (Pin_11), J1.2 (Pin_2)
Other:
- note added: "DMP"
- note added: "FLT"
- note added: "SCL"

Commit message: PCB layout
schematic finished, layout
Parts:
- removed J4: Output 1/4", Connector_Audio:Jack_6.35mm_Neutrik_NRJ6HM-1-PRE_Horizontal, symbol Connector_Audio:AudioJack2_Ground_Switch
- added J11: AudioJack3_Ground, Connector_Audio:Jack_6.35mm_Neutrik_NRJ3HF-1_Horizontal, symbol Connector_Audio:AudioJack3_Ground
Connections:
- net GND: now also J11.G, J11.S
- net OutputL: now also J11.T
- net OutputR: now also J11.R
Changed lines of the file:
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@@
+	(wire
+		(pts
+			(xy 209.55 83.82) (xy 204.47 83.82)
+		)
+		(stroke
+			(width 0)
+			(type default)
+		)
+	)
 	(wire
 		(pts
@@
 	(wire
 		(pts
+			(xy 204.47 83.82) (xy 204.47 71.12)
+		)
+		(stroke
+			(width 0)
+			(type default)
+		)
+	)
+	(wire
+		(pts
 			(xy 137.16 101.6) (xy 139.7 101.6)
 		)
@@
 	(wire
 		(pts
+			(xy 204.47 71.12) (xy 198.12 71.12)
+		)
+		(stroke
+			(width 0)
+			(type default)
+		)
+	)
+	(wire
+		(pts
 			(xy 173.99 99.06) (xy 173.99 91.44)
 		)
@@
 	(wire
 		(pts
-			(xy 204.47 99.06) (xy 204.47 91.44)
+			(xy 204.47 99.06) (xy 204.47 88.9)
 		)
 		(stroke
@@
 	(wire
 		(pts
-			(xy 204.47 91.44) (xy 207.01 91.44)
+			(xy 204.47 88.9) (xy 209.55 88.9)
 		)
 		(stroke
@@
 	(wire
 		(pts
-			(xy 198.12 86.36) (xy 207.01 86.36)
+			(xy 198.12 86.36) (xy 209.55 86.36)
 		)
 		(stroke
@@
 	)
 	(label "OutputL"
-		(at 207.01 91.44 180)
+		(at 207.01 88.9 180)
 		(effects
 			(font
@@
 	)
 	(symbol
+		(lib_id "Connector_Audio:AudioJack3_Ground")
+		(at 214.63 86.36 0)
+		(mirror y)
+		(unit 1)
+		(body_style 1)
+		(exclude_from_sim no)
+		(in_bom yes)
+		(on_board yes)
+		(in_pos_files yes)
+		(dnp no)
+		(property "Reference" "J11"
+			(at 216.535 77.47 0)
+			(show_name no)
+			(do_not_autoplace no)
+			(effects
+				(font
+					(size 1.27 1.27)
+				)
+			)
+		)
+		(property "Value" "AudioJack3_Ground"
+			(at 216.535 80.01 0)
+			(show_name no)
+			(do_not_autoplace no)
+			(effects
+				(font
+					(size 1.27 1.27)
+				)
+			)
+		)
+		(property "Footprint" "Connector_Audio:Jack_6.35mm_Neutrik_NRJ3HF-1_Horizontal"
+			(at 214.63 86.36 0)
+			(hide yes)
+			(show_name no)
+			(do_not_autoplace no)
+			(effects
+				(font
+					(size 1.27 1.27)
+				)
+			)
+		)
+		(property "Datasheet" ""
+			(at 214.63 86.36 0)
+			(hide yes)
+			(show_name no)
+			(do_not_autoplace no)
+			(effects
+				(font
+					(size 1.27 1.27)
+				)
+			)
+		)
+		(property "Description" "Audio Jack, 3 Poles (Stereo / TRS), Grounded Sleeve"
+			(at 214.63 86.36 0)
+			(hide yes)
+			(show_name no)
+			(do_not_autoplace no)
+			(effects
+				(font
+					(size 1.27 1.27)
+				)
+			)
+		)
+		(pin "T"
+		)
+		(pin "R"
+		)
+		(pin "S"
+		)
+		(pin "G"
+		)
+		(instances
+			(project "audiofx"
+				(path "/aae363e5-bb9b-4e8b-bcb3-9a42adce8813/6491a4aa-bc0c-4223-be67-2f04673d2b26"
+					(reference "J11")
+					(unit 1)
+				)
+			)
+		)
+	)
+	(symbol
 		(lib_id "power:+5VA")
 		(at 137.16 76.2 0)
@@
 	)
 	(symbol
-		(lib_id "Connector_Audio:AudioJack2_Ground_Switch")
-		(at 212.09 91.44 0)
-		(mirror y)
-		(unit 1)
-		(body_style 1)
-		(exclude_from_sim no)
-		(in_bom yes)
-		(on_board yes)
-		(in_pos_files yes)
-		(dnp no)
-		(property "Reference" "J4"
-			(at 212.725 80.01 0)
-			(show_name no)
-			(do_not_autoplace no)
-			(effects
-				(font
-					(size 1.27 1.27)
-				)
-			)
-		)
-		(property "Value" "Output 1/4\""
-			(at 212.725 82.55 0)
-			(show_name no)
-			(do_not_autoplace no)
-			(effects
-				(font
-					(size 1.27 1.27)
-				)
-			)
-		)
-		(property "Footprint" "Connector_Audio:Jack_6.35mm_Neutrik_NRJ6HM-1-PRE_Horizontal"
-			(at 212.09 86.36 0)
-			(hide yes)
-			(show_name no)
-			(do_not_autoplace no)
-			(effects
-				(font
-					(size 1.27 1.27)
-				)
-			)
-		)
-		(property "Datasheet" ""
-			(at 212.09 86.36 0)
-			(hide yes)
-			(show_name no)
-			(do_not_autoplace no)
-			(effects
-				(font
-					(size 1.27 1.27)
-				)
-			)
-		)
-		(property "Description" "Audio Jack, 2 Poles (Mono / TS), Grounded Sleeve, Switched Pole (Normalling)"
-			(at 212.09 91.44 0)
-			(hide yes)
-			(show_name no)
-			(do_not_autoplace no)
-			(effects
-				(font
-					(size 1.27 1.27)
-				)
-			)
-		)
-		(pin "S"
-		)
-		(pin "TN"
-		)
-		(pin "G"
-		)
-		(pin "SN"
-		)
-		(pin "T"
-		)
-		(instances
-			(project "audiofx"
-				(path "/aae363e5-bb9b-4e8b-bcb3-9a42adce8813/6491a4aa-bc0c-4223-be67-2f04673d2b26"
-					(reference "J4")
-					(unit 1)
-				)
-			)
-		)
-	)
-	(symbol
 		(lib_id "power:GND")
 		(at 177.8 88.9 0)
@@
 	(symbol
 		(lib_id "power:GND")
-		(at 212.09 99.06 0)
+		(at 198.12 71.12 0)
+		(unit 1)
+		(body_style 1)
+		(exclude_from_sim no)
+		(in_bom yes)
+		(on_board yes)
+		(in_pos_files yes)
+		(dnp no)
+		(fields_autoplaced yes)
+		(property "Reference" "#PWR060"
+			(at 198.12 77.47 0)
+			(hide yes)
+			(show_name no)
+			(do_not_autoplace no)
+			(effects
+				(font
+					(size 1.27 1.27)
+				)
+			)
+		)
+		(property "Value" "GND"
+			(at 198.12 76.2 0)
+			(show_name no)
+			(do_not_autoplace no)
+			(effects
+				(font
+					(size 1.27 1.27)
+				)
+			)
+		)
+		(property "Footprint" ""
+			(at 198.12 71.12 0)
+			(hide yes)
+			(show_name no)
+			(do_not_autoplace no)
+			(effects
+				(font
+					(size 1.27 1.27)
+				)
+			)
+		)
+		(property "Datasheet" ""
+			(at 198.12 71.12 0)
+			(hide yes)
+			(show_name no)
+			(do_not_autoplace no)
+			(effects
+				(font
+					(size 1.27 1.27)
+				)
+			)
+		)
+		(property "Description" "Power symbol creates a global label with name \"GND\" , ground"
+			(at 198.12 71.12 0)
+			(hide yes)
+			(show_name no)
+			(do_not_autoplace no)
+			(effects
+				(font
+					(size 1.27 1.27)
+				)
+			)
+		)
+		(pin "1"
+		)
+		(instances
+			(project "audiofx"
+				(path "/aae363e5-bb9b-4e8b-bcb3-9a42adce8813/6491a4aa-bc0c-4223-be67-2f04673d2b26"
+					(reference "#PWR060")
+					(unit 1)
+				)
+			)
+		)
+	)
+	(symbol
+		(lib_id "power:GND")
+		(at 214.63 93.98 0)
 		(unit 1)
 		(body_style 1)
@@
 		(fields_autoplaced yes)
 		(property "Reference" "#PWR024"
-			(at 212.09 105.41 0)
+			(at 214.63 100.33 0)
 			(hide yes)
 			(show_name no)
@@
 		)
 		(property "Value" "GND"
-			(at 212.09 104.14 0)
+			(at 214.63 99.06 0)
 			(show_name no)
 			(do_not_autoplace no)
@@
 		)
 		(property "Footprint" ""
-			(at 212.09 99.06 0)
+			(at 214.63 93.98 0)
 			(hide yes)
 			(show_name no)
@@
 		)
 		(property "Datasheet" ""
-			(at 212.09 99.06 0)
+			(at 214.63 93.98 0)
 			(hide yes)
 			(show_name no)
@@
 		)
 		(property "Description" "Power symbol creates a global label with name \"GND\" , ground"
-			(at 212.09 99.06 0)
-			(hide yes)
-			(show_name no)
+			(at 214.63 93.98 0)
+			(hide yes)
+			(show_name no)
