File: PSU.kicad_sch (KiCad schematic)
At the start: 0 parts

Commit message: PCB layout
schematic finished, layout
Parts:
- added C6, C7: GRM188Z71C475ME21D, Capacitor_SMD:C_0603_1608Metric_Pad1.08x0.95mm_HandSolder, symbol SamacSys_Parts:GRM188Z71C475ME21D
- added C8: 100 uF 16 V, Capacitor_THT:CP_Radial_D10.0mm_P5.00mm, symbol Device:C_Polarized
- added L1, L2: 82472C, Inductor_SMD:L_1210_3225Metric_Pad1.42x2.65mm_HandSolder, symbol SamacSys_Parts:82472C
- added PS1: CRE1S0505S3C, Connector:FanPinHeader_1x04_P2.54mm_Vertical, symbol SamacSys_Parts:CRE1S0505S3C
Connections:
- new net: L1.2, PS1.2 (+VIN)
- new net: L2.1, PS1.4 (+VOUT)
- new net +3.3V: C6.1, L1.1
- new net +5VA: C7.1, C8.1, L2.2
- new net GND: C6.2, C7.2, C8.2, PS1.1 (-VIN), PS1.3 (-VOUT)
