File: audiofx.kicad_sch (KiCad schematic)
At the start: 0 parts

Commit message: PCB layout
schematic finished, layout
Other:
- sheet ESP32 ports: added 17, 18/WS, 21, 43, 44; removed none
- sheet Input ports: added BCK, LRC, OUT, SCK; removed none
- sheet Output ports: added BCK, DIN, LCK; removed none
