File: input.kicad_sch (KiCad schematic)
At the start: 0 parts

Commit message: Preamp Created
J201 jfet
Parts:
- added C1: 47nF, Capacitor_THT:C_Disc_D3.0mm_W1.6mm_P2.50mm, symbol Device:C
- added C2, C3: 100nF, Capacitor_THT:C_Disc_D3.0mm_W1.6mm_P2.50mm, symbol Device:C
- added Q1: J201, Package_TO_SOT_THT:TO-92_HandSolder, symbol Device:Q_NJFET_GDS
- added R1: 10k 0.25W, Resistor_THT:R_Axial_DIN0204_L3.6mm_D1.6mm_P5.08mm_Horizontal, symbol Device:R
- added R2: 1Meg 0.25W, Resistor_THT:R_Axial_DIN0204_L3.6mm_D1.6mm_P5.08mm_Horizontal, symbol Device:R
Connections:
- new net: C1.2, Q1.1 (G), R2.1
- new net: C2.1, Q1.3 (S), R1.1
- new net +5VA: C3.1, Q1.2 (D)
- new net GND: C3.2, R1.2, R2.2
- new net PreampOut: C2.2

Commit message: Big changes! DAC, ADC, ESP32
schematic 80% complete
added pcm libary part of module maybe someone can use it :)
Parts:
- added C4: 100nF, Capacitor_THT:C_Disc_D3.0mm_W1.6mm_P2.50mm, symbol Device:C
- added C5: 1uF, Capacitor_SMD:C_0805_2012Metric_Pad1.18x1.45mm_HandSolder, symbol Device:C
- added J3: Input 1/4", Connector_Audio:Jack_6.35mm_Neutrik_NRJ6HM-1-PRE_Horizontal, symbol Connector_Audio:AudioJack2_Ground_Switch
- added M1: PCM1808, esp32:PCM1808, symbol esp32:PCM1808_M
- added R3, R4: 100R 0.25W, Resistor_THT:R_Axial_DIN0204_L3.6mm_D1.6mm_P5.08mm_Horizontal, symbol Device:R
Connections:
- net +5VA: now also R3.1, R4.1; no longer C3.1, Q1.2 (D)
- net GND: now also C4.2, C5.2, J3.G, J3.TN, M1.1 (FMY), M1.14 (GND), M1.16 (GND), M1.17 (GND), M1.18 (GND), M1.19 (GND), M1.2 (MD1), M1.3 (MD0), M1.4 (GND)
- net PreampOut: now also M1.9 (LIN)
- net InputT: now reaches C1.1
- net InputT: now also J3.T
- new net: C4.1, C5.1, M1.6 (5V), R4.2
- new net: C3.1, Q1.2 (D), R3.2
- new net +3.3V: M1.15 (3.3V)
- new net BCK: M1.10 (BCK)
- new net InputS: J3.S
- new net LRC: M1.12 (LRC)
- new net OUT: M1.11 (OUT)
- new net SCK: M1.13 (SCK)
Other:
- moved on the sheet: C1, C2, C3, Q1, R1, R2

Commit message: PCB layout
schematic finished, layout
Parts:
- removed J3: Input 1/4", Connector_Audio:Jack_6.35mm_Neutrik_NRJ6HM-1-PRE_Horizontal, symbol Connector_Audio:AudioJack2_Ground_Switch
- added J12: AudioJack3_Ground, Connector_Audio:Jack_6.35mm_Neutrik_NRJ3HF-1_Horizontal, symbol Connector_Audio:AudioJack3_Ground
Connections:
- net GND: now also J12.G, J12.S
- net InputT: now also J12.T
- new net InputR: J12.R
Changed lines of the file:
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@@
 	(wire
 		(pts
-			(xy 77.47 101.6) (xy 72.39 101.6)
+			(xy 69.85 104.14) (xy 77.47 104.14)
 		)
 		(stroke
@@
 	(wire
 		(pts
-			(xy 72.39 109.22) (xy 72.39 119.38)
+			(xy 72.39 101.6) (xy 72.39 119.38)
 		)
 		(stroke
@@
 	(wire
 		(pts
+			(xy 69.85 101.6) (xy 72.39 101.6)
+		)
+		(stroke
+			(width 0)
+			(type default)
+		)
+	)
+	(wire
+		(pts
 			(xy 185.42 100.33) (xy 185.42 102.87)
 		)
@@
 	(wire
 		(pts
-			(xy 67.31 114.3) (xy 67.31 119.38)
-		)
-		(stroke
-			(width 0)
-			(type default)
-		)
-	)
-	(wire
-		(pts
 			(xy 224.79 102.87) (xy 214.63 102.87)
 		)
@@
 	(wire
 		(pts
-			(xy 72.39 106.68) (xy 90.17 106.68)
+			(xy 69.85 106.68) (xy 90.17 106.68)
+		)
+		(stroke
+			(width 0)
+			(type default)
+		)
+	)
+	(wire
+		(pts
+			(xy 64.77 111.76) (xy 64.77 119.38)
 		)
 		(stroke
@@
 		)
 	)
-	(label "InputS"
-		(at 77.47 101.6 0)
+	(label "InputR"
+		(at 77.47 104.14 0)
 		(effects
 			(font
@@
 			)
 			(justify left)
-		)
-	)
-	(symbol
-		(lib_id "Connector_Audio:AudioJack2_Ground_Switch")
-		(at 67.31 106.68 0)
-		(unit 1)
-		(body_style 1)
-		(exclude_from_sim no)
-		(in_bom yes)
-		(on_board yes)
-		(in_pos_files yes)
-		(dnp no)
-		(fields_autoplaced yes)
-		(property "Reference" "J3"
-			(at 66.675 95.25 0)
-			(show_name no)
-			(do_not_autoplace no)
-			(effects
-				(font
-					(size 1.27 1.27)
-				)
-			)
-		)
-		(property "Value" "Input 1/4\""
-			(at 66.675 97.79 0)
-			(show_name no)
-			(do_not_autoplace no)
-			(effects
-				(font
-					(size 1.27 1.27)
-				)
-			)
-		)
-		(property "Footprint" "Connector_Audio:Jack_6.35mm_Neutrik_NRJ6HM-1-PRE_Horizontal"
-			(at 67.31 101.6 0)
-			(hide yes)
-			(show_name no)
-			(do_not_autoplace no)
-			(effects
-				(font
-					(size 1.27 1.27)
-				)
-			)
-		)
-		(property "Datasheet" ""
-			(at 67.31 101.6 0)
-			(hide yes)
-			(show_name no)
-			(do_not_autoplace no)
-			(effects
-				(font
-					(size 1.27 1.27)
-				)
-			)
-		)
-		(property "Description" "Audio Jack, 2 Poles (Mono / TS), Grounded Sleeve, Switched Pole (Normalling)"
-			(at 67.31 106.68 0)
-			(hide yes)
-			(show_name no)
-			(do_not_autoplace no)
-			(effects
-				(font
-					(size 1.27 1.27)
-				)
-			)
-		)
-		(pin "S"
-		)
-		(pin "TN"
-		)
-		(pin "G"
-		)
-		(pin "SN"
-		)
-		(pin "T"
-		)
-		(instances
-			(project "audiofx"
-				(path "/aae363e5-bb9b-4e8b-bcb3-9a42adce8813/c507a14d-d9d8-4e36-ae17-7075eb96f1b4"
-					(reference "J3")
-					(unit 1)
-				)
-			)
 		)
 	)
@@
 	)
 	(symbol
+		(lib_id "power:GND")
+		(at 64.77 119.38 0)
+		(mirror y)
+		(unit 1)
+		(body_style 1)
+		(exclude_from_sim no)
+		(in_bom yes)
+		(on_board yes)
+		(in_pos_files yes)
+		(dnp no)
+		(fields_autoplaced yes)
+		(property "Reference" "#PWR061"
+			(at 64.77 125.73 0)
+			(hide yes)
+			(show_name no)
+			(do_not_autoplace no)
+			(effects
+				(font
+					(size 1.27 1.27)
+				)
+			)
+		)
+		(property "Value" "GND"
+			(at 64.77 124.46 0)
+			(show_name no)
+			(do_not_autoplace no)
+			(effects
+				(font
+					(size 1.27 1.27)
+				)
+			)
+		)
+		(property "Footprint" ""
+			(at 64.77 119.38 0)
+			(hide yes)
+			(show_name no)
+			(do_not_autoplace no)
+			(effects
+				(font
+					(size 1.27 1.27)
+				)
+			)
+		)
+		(property "Datasheet" ""
+			(at 64.77 119.38 0)
+			(hide yes)
+			(show_name no)
+			(do_not_autoplace no)
+			(effects
+				(font
+					(size 1.27 1.27)
+				)
+			)
+		)
+		(property "Description" "Power symbol creates a global label with name \"GND\" , ground"
+			(at 64.77 119.38 0)
+			(hide yes)
+			(show_name no)
+			(do_not_autoplace no)
+			(effects
+				(font
+					(size 1.27 1.27)
+				)
+			)
+		)
+		(pin "1"
+		)
+		(instances
+			(project "audiofx"
+				(path "/aae363e5-bb9b-4e8b-bcb3-9a42adce8813/c507a14d-d9d8-4e36-ae17-7075eb96f1b4"
+					(reference "#PWR061")
+					(unit 1)
+				)
+			)
+		)
+	)
+	(symbol
 		(lib_id "Device:C")
 		(at 119.38 95.25 90)
@@
 				(path "/aae363e5-bb9b-4e8b-bcb3-9a42adce8813/c507a14d-d9d8-4e36-ae17-7075eb96f1b4"
 					(reference "C3")
+					(unit 1)
+				)
+			)
+		)
+	)
+	(symbol
+		(lib_id "Connector_Audio:AudioJack3_Ground")
+		(at 64.77 104.14 0)
+		(unit 1)
+		(body_style 1)
+		(exclude_from_sim no)
+		(in_bom yes)
+		(on_board yes)
+		(in_pos_files yes)
+		(dnp no)
+		(property "Reference" "J12"
+			(at 62.865 95.25 0)
+			(show_name no)
+			(do_not_autoplace no)
+			(effects
+				(font
+					(size 1.27 1.27)
+				)
+			)
+		)
+		(property "Value" "AudioJack3_Ground"
+			(at 62.865 97.79 0)
+			(show_name no)
+			(do_not_autoplace no)
+			(effects
+				(font
+					(size 1.27 1.27)
+				)
+			)
+		)
+		(property "Footprint" "Connector_Audio:Jack_6.35mm_Neutrik_NRJ3HF-1_Horizontal"
+			(at 64.77 104.14 0)
+			(hide yes)
+			(show_name no)
+			(do_not_autoplace no)
+			(effects
+				(font
+					(size 1.27 1.27)
+				)
+			)
+		)
+		(property "Datasheet" ""
+			(at 64.77 104.14 0)
+			(hide yes)
+			(show_name no)
+			(do_not_autoplace no)
+			(effects
+				(font
+					(size 1.27 1.27)
+				)
+			)
+		)
+		(property "Description" "Audio Jack, 3 Poles (Stereo / TRS), Grounded Sleeve"
+			(at 64.77 104.14 0)
+			(hide yes)
+			(show_name no)
+			(do_not_autoplace no)
+			(effects
+				(font
+					(size 1.27 1.27)
+				)
+			)
+		)
+		(pin "T"
+		)
+		(pin "R"
+		)
+		(pin "S"
+		)
+		(pin "G"
+		)
+		(instances
+			(project "audiofx"
+				(path "/aae363e5-bb9b-4e8b-bcb3-9a42adce8813/c507a14d-d9d8-4e36-ae17-7075eb96f1b4"
+					(reference "J12")
 					(unit 1)
 				)
@@
 					(unit 1)
 				)
-			)
-		)
-	)
-	(symbol
-		(lib_id "power:GND")
-		(at 67.31 119.38 0)
-		(unit 1)
-		(body_style 1)
-		(exclude_from_sim no)
-		(in_bom yes)
-		(on_board yes)
-		(in_pos_files yes)
-		(dnp no)
-		(fields_autoplaced yes)
-		(property "Reference" "#PWR022"
-			(at 67.31 125.73 0)
-			(hide yes)
-			(show_name no)
-			(do_not_autoplace no)
-			(effects
-				(font
-					(size 1.27 1.27)
-				)
-			)
-		)
-		(property "Value" "GND"
-			(at 67.31 124.46 0)
-			(show_name no)
-			(do_not_autoplace no)
-			(effects
-				(font
-					(size 1.27 1.27)
-				)
-			)
-		)
-		(property "Footprint" ""
-			(at 67.31 119.38 0)
-			(hide yes)
-			(show_name no)
-			(do_not_autoplace no)
-			(effects
-				(font
-					(size 1.27 1.27)
-				)
-			)
-		)
-		(property "Datasheet" ""
-			(at 67.31 119.38 0)
-			(hide yes)
-			(show_name no)
-			(do_not_autoplace no)
-			(effects
-				(font
-					(size 1.27 1.27)
-				)
-			)
-		)
-		(property "Description" "Power symbol creates a global label with name \"GND\" , ground"
-			(at 67.31 119.38 0)
-			(hide yes)
-			(show_name no)
-			(do_not_autoplace no)
-			(effects
-				(font
-					(size 1.27 1.27)
-				)
-			)
-		)
-		(pin "1"
-		)
-		(instances
-			(project "audiofx"
-				(path "/aae363e5-bb9b-4e8b-bcb3-9a42adce8813/c507a14d-d9d8-4e36-ae17-7075eb96f1b4"
-					(reference "#PWR022")
-					(unit 1)
-				)
